File: Throttle Control PCB/_autosave-Throttle Control PCB.sch (KiCad schematic (older format))
At the start: 20 parts

Commit message: Added the programmer pin header.
Parts:
- added D?: LED, symbol Device:LED
- added J?: Conn_02x03_Counter_Clockwise, symbol Connector_Generic:Conn_02x03_Counter_Clockwise
- added R?: 220, symbol Device:R
Connections:
- wire segments 70 -> 85
Other:
- moved on the sheet: C?, L?, R?, Y?
