File: Throttle Control PCB/Throttle Control PCB.sch (KiCad schematic (older format))
At the start: 14 parts

Commit message: Added +5V power supply.
Parts:
- added C?: 10μF, symbol Device:C
- added L?: 4.7μH, symbol Device:L
- added R?: 10k, symbol Device:R
- added U?: MCP1642D-50I_MS-ND, symbol Throttle~Control~Library:MCP1642D-50I_MS-ND
Connections:
- net labels added: +BATT
- wire segments 46 -> 62
Other:
- moved on the sheet: BT?
Changed lines of the file:
@@
-$EndComp
-$Comp
-L Device:Battery_Cell BT?
-U 1 1 5DA8BF17
-P 2450 1450
-F 0 "BT?" H 2568 1546 50  0000 L CNN
-F 1 "3.7V" H 2568 1455 50  0000 L CNN
-F 2 "" V 2450 1510 50  0001 C CNN
-F 3 "~" V 2450 1510 50  0001 C CNN
-	1    2450 1450
-	1    0    0    -1
 $EndComp
 $Comp
@@
 Wire Wire Line
 	7900 2200 7900 2250
+$Comp
+L Throttle~Control~Library:MCP1642D-50I_MS-ND U?
+U 1 1 5DAC5786
+P 2000 2150
+F 0 "U?" H 2025 2615 50  0000 C CNN
+F 1 "MCP1642D-50I_MS-ND" H 2025 2524 50  0000 C CNN
+F 2 "" H 1750 1800 50  0001 C CNN
+F 3 "" H 1750 1800 50  0001 C CNN
+	1    2000 2150
+	1    0    0    -1
+$EndComp
+$Comp
+L power:GND #PWR?
+U 1 1 5DAC67E6
+P 2650 2100
+F 0 "#PWR?" H 2650 1850 50  0001 C CNN
+F 1 "GND" H 2655 1927 50  0000 C CNN
+F 2 "" H 2650 2100 50  0001 C CNN
+F 3 "" H 2650 2100 50  0001 C CNN
+	1    2650 2100
+	1    0    0    -1
+$EndComp
+Wire Wire Line
+	2400 2250 2500 2250
+Wire Wire Line
+	2400 2100 2500 2100
+Wire Wire Line
+	2500 2100 2500 2250
+$Comp
+L power:GND #PWR?
+U 1 1 5DAD21D0
+P 1300 1250
+F 0 "#PWR?" H 1300 1000 50  0001 C CNN
+F 1 "GND" H 1305 1077 50  0000 C CNN
+F 2 "" H 1300 1250 50  0001 C CNN
+F 3 "" H 1300 1250 50  0001 C CNN
+	1    1300 1250
+	1    0    0    -1
+$EndComp
+$Comp
+L Device:Battery_Cell BT?
+U 1 1 5DA8BF17
+P 1300 1150
+F 0 "BT?" H 1000 1250 50  0000 L CNN
+F 1 "3.7V" H 1000 1150 50  0000 L CNN
+F 2 "" V 1300 1210 50  0001 C CNN
+F 3 "~" V 1300 1210 50  0001 C CNN
+	1    1300 1150
+	1    0    0    -1
+$EndComp
+$Comp
+L power:+BATT #PWR?
+U 1 1 5DAE0380
+P 2500 1750
+F 0 "#PWR?" H 2500 1600 50  0001 C CNN
+F 1 "+BATT" H 2515 1923 50  0000 C CNN
+F 2 "" H 2500 1750 50  0001 C CNN
+F 3 "" H 2500 1750 50  0001 C CNN
+	1    2500 1750
+	1    0    0    -1
+$EndComp
+Wire Wire Line
+	2500 1750 2500 1950
+Wire Wire Line
+	2500 1950 2400 1950
+$Comp
+L power:+5V #PWR?
+U 1 1 5DAE2C88
+P 1250 2300
+F 0 "#PWR?" H 1250 2150 50  0001 C CNN
+F 1 "+5V" H 1265 2473 50  0000 C CNN
+F 2 "" H 1250 2300 50  0001 C CNN
+F 3 "" H 1250 2300 50  0001 C CNN
+	1    1250 2300
+	1    0    0    -1
+$EndComp
+Wire Wire Line
+	1250 2300 1250 2400
+Wire Wire Line
+	1250 2400 1650 2400
+$Comp
+L power:+BATT #PWR?
+U 1 1 5DACF02C
+P 1300 800
+F 0 "#PWR?" H 1300 650 50  0001 C CNN
+F 1 "+BATT" H 1315 973 50  0000 C CNN
+F 2 "" H 1300 800 50  0001 C CNN
+F 3 "" H 1300 800 50  0001 C CNN
+	1    1300 800
+	1    0    0    -1
+$EndComp
+$Comp
+L Device:C C?
+U 1 1 5DAE87CD
+P 1600 900
+F 0 "C?" V 1348 900 50  0000 C CNN
+F 1 "10μF" V 1439 900 50  0000 C CNN
+F 2 "" H 1638 750 50  0001 C CNN
+F 3 "~" H 1600 900 50  0001 C CNN
+	1    1600 900
+	0    1    1    0
+$EndComp
+Wire Wire Line
+	1450 900  1300 900
+Wire Wire Line
+	1300 800  1300 900
+Connection ~ 1300 900
+Wire Wire Line
+	1300 900  1300 950
+$Comp
+L power:GND #PWR?
+U 1 1 5DAEA1A3
+P 1750 1250
+F 0 "#PWR?" H 1750 1000 50  0001 C CNN
+F 1 "GND" H 1755 1077 50  0000 C CNN
+F 2 "" H 1750 1250 50  0001 C CNN
+F 3 "" H 1750 1250 50  0001 C CNN
+	1    1750 1250
+	1    0    0    -1
+$EndComp
+Wire Wire Line
+	1750 900  1750 1250
+$Comp
+L Device:R R?
+U 1 1 5DAEDB4C
+P 1400 1800
+F 0 "R?" H 1470 1846 50  0000 L CNN
+F 1 "10k" H 1470 1755 50  0000 L CNN
+F 2 "" V 1330 1800 50  0001 C CNN
+F 3 "~" H 1400 1800 50  0001 C CNN
+	1    1400 1800
+	1    0    0    -1
+$EndComp
+$Comp
+L power:+BATT #PWR?
+U 1 1 5DAEE9CD
+P 1400 1650
+F 0 "#PWR?" H 1400 1500 50  0001 C CNN
+F 1 "+BATT" H 1415 1823 50  0000 C CNN
+F 2 "" H 1400 1650 50  0001 C CNN
+F 3 "" H 1400 1650 50  0001 C CNN
+	1    1400 1650
+	1    0    0    -1
+$EndComp
+Wire Wire Line
+	1400 1950 1650 1950
+$Comp
+L Device:L L?
+U 1 1 5DAF1C3F
+P 2700 2400
+F 0 "L?" V 2519 2400 50  0000 C CNN
+F 1 "4.7μH" V 2610 2400 50  0000 C CNN
+F 2 "" H 2700 2400 50  0001 C CNN
+F 3 "~" H 2700 2400 50  0001 C CNN
+	1    2700 2400
+	0    -1   -1   0
+$EndComp
+Wire Wire Line
+	2500 2100 2650 2100
+Connection ~ 2500 2100
+Wire Wire Line
+	2400 2400 2550 2400
+$Comp
+L power:+BATT #PWR?
+U 1 1 5DAFF791
+P 2900 2200
+F 0 "#PWR?" H 2900 2050 50  0001 C CNN
+F 1 "+BATT" H 2915 2373 50  0000 C CNN
+F 2 "" H 2900 2200 50  0001 C CNN
+F 3 "" H 2900 2200 50  0001 C CNN
+	1    2900 2200
+	1    0    0    -1
+$EndComp
+Wire Wire Line
+	2850 2400 2900 2400
+Wire Wire Line
+	2900 2400 2900 2200
 $EndSCHEMATC

Commit message: Connected RJ45 to CAN transciever.
Parts:
- added JP?: SolderJumper_2_Open, symbol Jumper:SolderJumper_2_Open
- added R?: 120, symbol Device:R
- C? (x4): value 10pF -> 20pF
- Y?: value 8MHz? -> 16MHz
Connections:
- wire segments 62 -> 70
Other:
- moved on the sheet: J?, L?, R?
Changed lines of the file:
@@
 P 4400 4300
 F 0 "C?" V 4550 4300 50  0000 C CNN
-F 1 "10pF" V 4650 4300 50  0000 C CNN
+F 1 "20pF" V 4650 4300 50  0000 C CNN
 F 2 "" H 4438 4150 50  0001 C CNN
 F 3 "~" H 4400 4300 50  0001 C CNN
@@
 P 4700 4300
 F 0 "C?" V 4952 4300 50  0000 C CNN
-F 1 "10pF" V 4861 4300 50  0000 C CNN
+F 1 "20pF" V 4861 4300 50  0000 C CNN
 F 2 "" H 4738 4150 50  0001 C CNN
 F 3 "~" H 4700 4300 50  0001 C CNN
@@
 L Connector:RJ45 J?
 U 1 1 5DA7E49C
-P 7300 4950
-F 0 "J?" H 6970 4954 50  0000 R CNN
-F 1 "RJ45" H 6970 5045 50  0000 R CNN
-F 2 "" V 7300 4975 50  0001 C CNN
-F 3 "~" V 7300 4975 50  0001 C CNN
-	1    7300 4950
-	-1   0    0    1
+P 7500 4900
+F 0 "J?" H 7170 4904 50  0000 R CNN
+F 1 "RJ45" H 7170 4995 50  0000 R CNN
+F 2 "" V 7500 4925 50  0001 C CNN
+F 3 "~" V 7500 4925 50  0001 C CNN
+	1    7500 4900
+	0    -1   -1   0
 $EndComp
 $Comp
@@
 P 5050 3250
 F 0 "Y?" H 5000 3100 50  0000 L CNN
-F 1 "8MHz?" H 4900 3000 50  0000 L CNN
+F 1 "16MHz" H 4900 3000 50  0000 L CNN
 F 2 "" H 5050 3250 50  0001 C CNN
 F 3 "~" H 5050 3250 50  0001 C CNN
@@
 P 4900 3400
 F 0 "C?" H 5000 3300 50  0000 C CNN
-F 1 "10pF" H 5050 3200 50  0000 C CNN
+F 1 "20pF" H 5050 3200 50  0000 C CNN
 F 2 "" H 4938 3250 50  0001 C CNN
 F 3 "~" H 4900 3400 50  0001 C CNN
@@
 P 5200 3400
 F 0 "C?" V 5452 3400 50  0000 C CNN
-F 1 "10pF" V 5361 3400 50  0000 C CNN
+F 1 "20pF" V 5361 3400 50  0000 C CNN
 F 2 "" H 5238 3250 50  0001 C CNN
 F 3 "~" H 5200 3400 50  0001 C CNN
@@
 L Throttle~Control~Library:MCP1642D-50I_MS-ND U?
 U 1 1 5DAC5786
-P 2000 2150
-F 0 "U?" H 2025 2615 50  0000 C CNN
-F 1 "MCP1642D-50I_MS-ND" H 2025 2524 50  0000 C CNN
-F 2 "" H 1750 1800 50  0001 C CNN
-F 3 "" H 1750 1800 50  0001 C CNN
-	1    2000 2150
+P 3550 1250
+F 0 "U?" H 3575 1715 50  0000 C CNN
+F 1 "MCP1642D-50I_MS-ND" H 3575 1624 50  0000 C CNN
+F 2 "" H 3300 900 50  0001 C CNN
+F 3 "" H 3300 900 50  0001 C CNN
+	1    3550 1250
 	1    0    0    -1
 $EndComp
@@
 L power:GND #PWR?
 U 1 1 5DAC67E6
-P 2650 2100
-F 0 "#PWR?" H 2650 1850 50  0001 C CNN
-F 1 "GND" H 2655 1927 50  0000 C CNN
-F 2 "" H 2650 2100 50  0001 C CNN
-F 3 "" H 2650 2100 50  0001 C CNN
-	1    2650 2100
-	1    0    0    -1
-$EndComp
-Wire Wire Line
-	2400 2250 2500 2250
-Wire Wire Line
-	2400 2100 2500 2100
-Wire Wire Line
-	2500 2100 2500 2250
+P 4200 1200
+F 0 "#PWR?" H 4200 950 50  0001 C CNN
+F 1 "GND" H 4205 1027 50  0000 C CNN
+F 2 "" H 4200 1200 50  0001 C CNN
+F 3 "" H 4200 1200 50  0001 C CNN
+	1    4200 1200
+	1    0    0    -1
+$EndComp
+Wire Wire Line
+	3950 1350 4050 1350
+Wire Wire Line
+	3950 1200 4050 1200
+Wire Wire Line
+	4050 1200 4050 1350
 $Comp
 L power:GND #PWR?
@@
 L power:+BATT #PWR?
 U 1 1 5DAE0380
-P 2500 1750
-F 0 "#PWR?" H 2500 1600 50  0001 C CNN
-F 1 "+BATT" H 2515 1923 50  0000 C CNN
-F 2 "" H 2500 1750 50  0001 C CNN
-F 3 "" H 2500 1750 50  0001 C CNN
-	1    2500 1750
-	1    0    0    -1
-$EndComp
-Wire Wire Line
-	2500 1750 2500 1950
-Wire Wire Line
-	2500 1950 2400 1950
-$Comp
-L power:+5V #PWR?
-U 1 1 5DAE2C88
-P 1250 2300
-F 0 "#PWR?" H 1250 2150 50  0001 C CNN
-F 1 "+5V" H 1265 2473 50  0000 C CNN
-F 2 "" H 1250 2300 50  0001 C CNN
-F 3 "" H 1250 2300 50  0001 C CNN
-	1    1250 2300
-	1    0    0    -1
-$EndComp
-Wire Wire Line
-	1250 2300 1250 2400
-Wire Wire Line
-	1250 2400 1650 2400
+P 4050 850
+F 0 "#PWR?" H 4050 700 50  0001 C CNN
+F 1 "+BATT" H 4065 1023 50  0000 C CNN
+F 2 "" H 4050 850 50  0001 C CNN
+F 3 "" H 4050 850 50  0001 C CNN
+	1    4050 850
+	1    0    0    -1
+$EndComp
+Wire Wire Line
+	4050 850  4050 1050
+Wire Wire Line
+	4050 1050 3950 1050
 $Comp
 L power:+BATT #PWR?
@@
 L Device:R R?
 U 1 1 5DAEDB4C
-P 1400 1800
-F 0 "R?" H 1470 1846 50  0000 L CNN
-F 1 "10k" H 1470 1755 50  0000 L CNN
-F 2 "" V 1330 1800 50  0001 C CNN
-F 3 "~" H 1400 1800 50  0001 C CNN
-	1    1400 1800
+P 2950 900
+F 0 "R?" H 3020 946 50  0000 L CNN
+F 1 "10k" H 3020 855 50  0000 L CNN
+F 2 "" V 2880 900 50  0001 C CNN
+F 3 "~" H 2950 900 50  0001 C CNN
+	1    2950 900
 	1    0    0    -1
 $EndComp
@@
 L power:+BATT #PWR?
 U 1 1 5DAEE9CD
-P 1400 1650
-F 0 "#PWR?" H 1400 1500 50  0001 C CNN
-F 1 "+BATT" H 1415 1823 50  0000 C CNN
-F 2 "" H 1400 1650 50  0001 C CNN
-F 3 "" H 1400 1650 50  0001 C CNN
-	1    1400 1650
-	1    0    0    -1
-$EndComp
-Wire Wire Line
-	1400 1950 1650 1950
+P 2950 750
+F 0 "#PWR?" H 2950 600 50  0001 C CNN
+F 1 "+BATT" H 2965 923 50  0000 C CNN
+F 2 "" H 2950 750 50  0001 C CNN
+F 3 "" H 2950 750 50  0001 C CNN
+	1    2950 750
+	1    0    0    -1
+$EndComp
+Wire Wire Line
+	2950 1050 3200 1050
 $Comp
 L Device:L L?
 U 1 1 5DAF1C3F
-P 2700 2400
-F 0 "L?" V 2519 2400 50  0000 C CNN
-F 1 "4.7μH" V 2610 2400 50  0000 C CNN
-F 2 "" H 2700 2400 50  0001 C CNN
-F 3 "~" H 2700 2400 50  0001 C CNN
-	1    2700 2400
+P 4250 1500
+F 0 "L?" V 4069 1500 50  0000 C CNN
+F 1 "4.7μH" V 4160 1500 50  0000 C CNN
+F 2 "" H 4250 1500 50  0001 C CNN
+F 3 "~" H 4250 1500 50  0001 C CNN
+	1    4250 1500
 	0    -1   -1   0
 $EndComp
 Wire Wire Line
-	2500 2100 2650 2100
-Connection ~ 2500 2100
-Wire Wire Line
-	2400 2400 2550 2400
+	4050 1200 4200 1200
+Connection ~ 4050 1200
+Wire Wire Line
+	3950 1500 4100 1500
 $Comp
 L power:+BATT #PWR?
 U 1 1 5DAFF791
-P 2900 2200
-F 0 "#PWR?" H 2900 2050 50  0001 C CNN
-F 1 "+BATT" H 2915 2373 50  0000 C CNN
-F 2 "" H 2900 2200 50  0001 C CNN
-F 3 "" H 2900 2200 50  0001 C CNN
-	1    2900 2200
-	1    0    0    -1
-$EndComp
-Wire Wire Line
-	2850 2400 2900 2400
-Wire Wire Line
-	2900 2400 2900 2200
+P 4450 1300
+F 0 "#PWR?" H 4450 1150 50  0001 C CNN
+F 1 "+BATT" H 4465 1473 50  0000 C CNN
+F 2 "" H 4450 1300 50  0001 C CNN
+F 3 "" H 4450 1300 50  0001 C CNN
+	1    4450 1300
+	1    0    0    -1
+$EndComp
+Wire Wire Line
+	4400 1500 4450 1500
+Wire Wire Line
+	4450 1500 4450 1300
+Wire Wire Line
+	2800 1500 3200 1500
+Wire Wire Line
+	2800 1400 2800 1500
+$Comp
+L power:+5V #PWR?
+U 1 1 5DAE2C88
+P 2800 1400
+F 0 "#PWR?" H 2800 1250 50  0001 C CNN
+F 1 "+5V" H 2815 1573 50  0000 C CNN
+F 2 "" H 2800 1400 50  0001 C CNN
+F 3 "" H 2800 1400 50  0001 C CNN
+	1    2800 1400
+	1    0    0    -1
+$EndComp
+Wire Wire Line
+	7600 3250 7600 3450
+$Comp
+L Jumper:SolderJumper_2_Open JP?
+U 1 1 5DAFBD6A
+P 7050 3600
+F 0 "JP?" V 7004 3668 50  0000 L CNN
+F 1 "SolderJumper_2_Open" V 7095 3668 50  0000 L CNN
+F 2 "" H 7050 3600 50  0001 C CNN
+F 3 "~" H 7050 3600 50  0001 C CNN
+	1    7050 3600
+	0    1    1    0
+$EndComp
+$Comp
+L Device:R R?
+U 1 1 5DAFD8A6
+P 7050 3900
+F 0 "R?" H 7120 3946 50  0000 L CNN
+F 1 "120" H 7120 3855 50  0000 L CNN
+F 2 "" V 6980 3900 50  0001 C CNN
+F 3 "~" H 7050 3900 50  0001 C CNN
+	1    7050 3900
+	1    0    0    -1
+$EndComp
+Wire Wire Line
+	7800 3250 7800 4050
+Wire Wire Line
+	7600 3450 7050 3450
+Connection ~ 7600 3450
+Wire Wire Line
+	7050 4050 7800 4050
+Connection ~ 7800 4050
+Wire Wire Line
+	7800 4050 7800 4500
+Wire Wire Line
+	7600 4400 7700 4400
+Wire Wire Line
+	7700 4400 7700 4500
+Wire Wire Line
+	7600 3450 7600 4400
 $EndSCHEMATC

Commit message: Prepared connection headers for the 12V power supply board.
Parts:
- added D?: LED, symbol Device:LED
- added J?: Conn_02x03_Counter_Clockwise, symbol Connector_Generic:Conn_02x03_Counter_Clockwise
- added J?: Conn_01x06, symbol Connector_Generic:Conn_01x06
- added R?: 220, symbol Device:R
Connections:
- net labels added: +12V
- wire segments 70 -> 96
Other:
- note added: "Connects to the boost converter daughter-board."
- note added: "Programmer input"
- moved on the sheet: C?, J?, JP?, L?, R?, U?, Y?

Commit message: Added pinouts for servos and servo circuitry
Parts:
- removed J?: Conn_01x06, symbol Connector_Generic:Conn_01x06
- added C? (x2): C, symbol Device:C
- added D?: D_Schottky, symbol Device:D_Schottky
- added J?: Screw_Terminal_01x02, symbol Connector:Screw_Terminal_01x02
- added J?: Limit Switch, symbol Connector_Generic:Conn_01x02
- added J?: Ball Servo 1, symbol Connector_Generic:Conn_01x03
- added J?: Pressure Transducer, symbol Connector:Screw_Terminal_01x03
- added J?: Ball Servo 2, symbol Connector_Generic:Conn_01x03
- added J?: Continuous Rotation Servo, symbol Connector_Generic:Conn_01x04
- added L?: L, symbol Device:L
- added R?: 900, symbol Device:R
- added R?: 1k, symbol Device:R
- added RV?: R_POT_TRIM, symbol Device:R_POT_TRIM
- added U?: MAX6675, symbol Throttle~Control~Library:MAX6675
- added U?: MT3608, symbol iclr:MT3608
Connections:
- net labels added: +6V, ENC1, PT, RST, S1, S2, S3, SCK, SI, SO
- net labels removed: +12V
- wire segments 96 -> 144
Other:
- note removed: "Connects to the boost converter daughter-board."
- moved on the sheet: C?, J?, R?, Y?

Commit message: Added pressure transducer
Parts:
- added C?: 22μF, symbol Device:C
- C?: value 10μF -> 22μF
- C? (x2): value C -> 22μF
Connections:
- wire segments 144 -> 148
Other:
- moved on the sheet: C?, D?, J?, L?, R?, RV?, U?
